File: PCB_SALUS_v2.kicad_sch (KiCad schematic)
At the start: 0 parts

Commit message: Added IMU
Other:
- added sheet SENSORES (SENSORES.kicad_sch)
Changed lines of the file:
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@@
+	)
+	(sheet
+		(at 162.56 24.13)
+		(size 48.26 38.1)
+		(exclude_from_sim no)
+		(in_bom yes)
+		(on_board yes)
+		(dnp no)
+		(fields_autoplaced yes)
+		(stroke
+			(width 0.1524)
+			(type solid)
+		)
+		(fill
+			(color 0 0 0 0)
+		)
+		(property "Sheetname" "SENSORES"
+			(at 162.56 23.4184 0)
+			(show_name no)
+			(do_not_autoplace no)
+			(effects
+				(font
+					(size 1.27 1.27)
+				)
+				(justify left bottom)
+			)
+		)
+		(property "Sheetfile" "SENSORES.kicad_sch"
+			(at 162.56 62.8146 0)
+			(show_name no)
+			(do_not_autoplace no)
+			(effects
+				(font
+					(size 1.27 1.27)
+				)
+				(justify left top)
+			)
+		)
+		(instances
+			(project "PCB_SALUS_v2"
+				(path "/73bd63ea-8f0f-4b31-8d24-3cde4b540ad9"
+					(page "4")
+				)
+			)
+		)
 	)
 	(sheet

Commit message: Added IMU
Other:
- removed sheet ALIMENTACION
Changed lines of the file:
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@@
-		)
-	)
-	(sheet
-		(at 24.13 20.32)
-		(size 41.91 36.83)
-		(exclude_from_sim no)
-		(in_bom yes)
-		(on_board yes)
-		(dnp no)
-		(fields_autoplaced yes)
-		(stroke
-			(width 0.1524)
-			(type solid)
-		)
-		(fill
-			(color 0 0 0 0)
-		)
-		(property "Sheetname" "ALIMENTACION"
-			(at 24.13 19.6084 0)
-			(show_name no)
-			(do_not_autoplace no)
-			(effects
-				(font
-					(size 1.27 1.27)
-				)
-				(justify left bottom)
-			)
-		)
-		(property "Sheetfile" "01_ALIMENTACION.kicad_sch"
-			(at 24.13 57.7346 0)
-			(show_name no)
-			(do_not_autoplace no)
-			(effects
-				(font
-					(size 1.27 1.27)
-				)
-				(justify left top)
-			)
-		)
-		(instances
-			(project "PCB_SALUS_v2"
-				(path "/73bd63ea-8f0f-4b31-8d24-3cde4b540ad9"
-					(page "2")
-				)
-			)
 		)
 	)
