File: ESP32.kicad_sch (KiCad schematic)
At the start: 32 parts, among them J1 Conn_01x06, J3 USB_C_Receptacle_USB2.0_16P, Q3 SS8050, Q4 SS8050, U1 TLV75733PDBV, U2 ESP32-WROOM-32E, U3 CP2102N-A02-GQFN24

Commit message: Added IMU
Parts:
- added J4: Conn_01x03, symbol Connector_Generic:Conn_01x03
- added J5: Jack-DC, symbol Connector:Jack-DC
- added R11, R12: 1k, symbol Device:R
- C1, C10, C3, C5, C7: footprint (none) -> Capacitor_SMD:C_0805_2012Metric
- C11, C2, C4, C6, C9: footprint (none) -> Capacitor_SMD:C_0603_1608Metric
- C8: value 100nF -> 10uF
- J1: footprint (none) -> Connector_PinHeader_2.54mm:PinHeader_1x06_P2.54mm_Vertical
- J3: footprint (none) -> Connector_USB:USB_C_Receptacle_G-Switch_GT-USB-7010ASV
- R10, R4, R5, R6, R7, R8, R9: footprint (none) -> Resistor_SMD:R_0603_1608Metric
Connections:
- net +5V: now also J5.2
- net GND: now also J4.3 (Pin_3), J5.1
- net CS_ACCEL: now reaches U2.10 (IO25)
- net CS_GIRO: now reaches U2.11 (IO26)
- net at U2.27 (IO16): now also R11.2
- net at U2.28 (IO17): now also R12.2
- net SPI_CLOCK: now reaches U2.30 (IO18)
- net SPI_MISO: now reaches U2.31 (IO19)
- net SPI_MOSI: now reaches U2.37 (IO23)
- net DR_ACCEL: now reaches U2.6 (IO34)
- net DR_GIRO: now reaches U2.7 (IO35)
- new net U1_RX: J4.2 (Pin_2), R11.1
- new net U1_TX: J4.1 (Pin_1), R12.1
Other:
- note added: "5V INPUT"
- note added: "UART1"
- moved on the sheet: C10, C11, C7, C9, Q3, Q4, R10, R6, R7, R8, R9, U2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

Commit message: Added IMU
Parts:
- C1, C3, C5: LCSC PN (none) -> C17024; MPN (none) -> CL21A106KPFNNNE; Manufacturer (none) -> Samsung Electro-Mechanics; Manufacturer Part (none) -> CL21A106KPFNNNE
- C10, C7: LCSC PN (none) -> C107125; MPN (none) -> CC0805KKX5R6BB475; Manufacturer (none) -> YAGEO; Manufacturer Part (none) -> CC0805KKX5R6BB475
- C11, C2, C4, C6, C9: LCSC PN (none) -> C1590; MPN (none) -> CL10B104KA8NNNC; Manufacturer (none) -> Samsung Electro-Mechanics; Manufacturer Part (none) -> CL10B104KA8NNNC
- C8: footprint Capacitor_SMD:C_0603_1608Metric -> Capacitor_SMD:C_0805_2012Metric; LCSC PN C1590 -> C17024; MPN (none) -> CL21A106KPFNNNE; Manufacturer (none) -> Samsung Electro-Mechanics; Manufacturer Part (none) -> CL21A106KPFNNNE
- D2: LCSC PN (none) -> C3040626; MPN (none) -> SP0503BAHTG; Manufacturer (none) -> Littelfuse; Manufacturer Part (none) -> SP0503BAHTG
- D3, D4: LCSC PN (none) -> C2480; MPN (none) -> SS14; Manufacturer (none) -> Yangzhou Yangjie Electronic Technology; Manufacturer Part (none) -> SS14
- J1: footprint Connector_PinHeader_2.54mm:PinHeader_1x06_P2.54mm_Vertical -> Connector_JST:JST_XH_S6B-XH-SM4-TB_1x06-1MP_P2.50mm_Horizontal; BOM Comments (none) -> Conector SMD de programacion; requiere housing XHP-6 y term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; LCSC PN (none) -> C20493992; MPN (none) -> S6B-XH-SM4-TB(LF)(SN); Manufacturer (none) -> JST; Manufacturer Part (none) -> S6B-XH-SM4-TB(LF)(SN)
- J3: LCSC PN (none) -> C2988369; MPN (none) -> GT-USB-7010ASV; Manufacturer (none) -> G-Switch; Manufacturer Part (none) -> GT-USB-7010ASV
- J4: footprint (none) -> Connector_JST:JST_XH_S3B-XH-SM4-TB_1x03-1MP_P2.50mm_Horizontal; BOM Comments (none) -> Conector SMD de 3 pines; requiere housing XHP-3 y terminale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; LCSC PN (none) -> C5306495; MPN (none) -> S3B-XH-SM4-TB(LF)(SN); Manufacturer (none) -> JST; Manufacturer Part (none) -> S3B-XH-SM4-TB(LF)(SN)
- J5: BOM Comments (none) -> NO MONTAR. Entrada de alimentacion pendiente; sin huella ni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; now not fitted; now left out of the parts list
- Q3, Q4: LCSC PN (none) -> C2150; MPN (none) -> SS8050; Manufacturer (none) -> Changjiang Electronics Technology (CJ); Manufacturer Part (none) -> SS8050
- R10: LCSC PN (none) -> C21190; MPN (none) -> 0603WAF1001T5E; Manufacturer (none) -> UNI-ROYAL(Uniroyal Elec); Manufacturer Part (none) -> 0603WAF1001T5E
- R11, R12: footprint (none) -> Resistor_SMD:R_0603_1608Metric; LCSC PN (none) -> C21190; MPN (none) -> 0603WAF1001T5E; Manufacturer (none) -> UNI-ROYAL(Uniroyal Elec); Manufacturer Part (none) -> 0603WAF1001T5E
- R22, R23: value 10K -> 10k; LCSC PN C98220 -> C25804; MPN (none) -> 0603WAF1002T5E; Manufacturer (none) -> UNI-ROYAL(Uniroyal Elec); Manufacturer Part (none) -> 0603WAF1002T5E
- R4, R5: LCSC PN (none) -> C23186; MPN (none) -> 0603WAF5101T5E; Manufacturer (none) -> UNI-ROYAL(Uniroyal Elec); Manufacturer Part (none) -> 0603WAF5101T5E
- R6: LCSC PN (none) -> C25961; MPN (none) -> 0603WAF2212T5E; Manufacturer (none) -> UNI-ROYAL(Uniroyal Elec); Manufacturer Part (none) -> 0603WAF2212T5E
- R7: LCSC PN (none) -> C23061; MPN (none) -> 0603WAF4752T5E; Manufacturer (none) -> UNI-ROYAL(Uniroyal Elec); Manufacturer Part (none) -> 0603WAF4752T5E
- R8, R9: LCSC PN (none) -> C25804; MPN (none) -> 0603WAF1002T5E; Manufacturer (none) -> UNI-ROYAL(Uniroyal Elec); Manufacturer Part (none) -> 0603WAF1002T5E
- SW1, SW2: MPN (none) -> TS1201-TZ25HAM
- U1: LCSC PN (none) -> C485517; MPN (none) -> TLV75733PDBVR; Manufacturer (none) -> Texas Instruments; Manufacturer Part (none) -> TLV75733PDBVR
- U2: LCSC PN (none) -> C701342; MPN (none) -> ESP32-WROOM-32E-N8; Manufacturer (none) -> Espressif Systems; Manufacturer Part (none) -> ESP32-WROOM-32E-N8
- U3: LCSC PN (none) -> C969151; MPN (none) -> CP2102N-A02-GQFN24R; Manufacturer (none) -> Silicon Labs; Manufacturer Part (none) -> CP2102N-A02-GQFN24R

Commit message: Esquematico preparado para revision
Parts:
- added R20: 10k, symbol Device:R
Connections:
- net CS_ACCEL: now also U2.26 (IO4); no longer U2.10 (IO25)
- net GND: now also R20.1
- net R_PWM: now reaches U2.12 (IO27)
- net RELAY_OE: now reaches U2.13 (IO14)
- net RELAY_LATCH: now reaches U2.14 (IO12)
- net RELAY_LATCH: now also R20.2
- net HALL_B: now reaches U2.16 (IO13)
- net HALL_C: now reaches U2.23 (IO15)
- net HALL_A: now reaches U2.29 (IO5)
- net I2C_SDA: now reaches U2.33 (IO21)
- net I2C_SCL: now reaches U2.36 (IO22)
- net FC_LEFT: now reaches U2.4 (SENSOR_VP)
- net FC_RIGHT: now reaches U2.5 (SENSOR_VN)
- net RF_PPM: now reaches U2.8 (IO32)
- net L_PWM: now reaches U2.9 (IO33)
- new net DAC: U2.10 (IO25)
Other:
- moved on the sheet: R11, R12, U2

Commit message: Schematic complete and ERC clean
Parts:
- removed J5: Jack-DC, symbol Connector:Jack-DC
- added J5: Conn_01x02, Connector_PinHeader_2.54mm:PinHeader_1x02_P2.54mm_Vertical, symbol Connector_Generic:Conn_01x02
- J1: value Conn_01x06 -> Header_THT_1x06_P2.54mm; footprint Connector_JST:JST_XH_S6B-XH-SM4-TB_1x06-1MP_P2.50mm_Horizontal -> Connector_PinHeader_2.54mm:PinHeader_1x06_P2.54mm_Vertical; BOM Comments Conector SMD de programacion; requiere housing XHP-6 y term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 -> Montaje manual: header THT vertical 1x06, paso 2.54 mm. Exc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; LCSC PN C20493992 -> (none); MPN S6B-XH-SM4-TB(LF)(SN) -> Header generico THT 1x06 P2.54 mm; Manufacturer JST -> Compra manual; Manufacturer Part S6B-XH-SM4-TB(LF)(SN) -> Header generico THT 1x06, P2.54 mm, vertical
- J4: value Conn_01x03 -> Header_THT_1x03_P2.54mm; footprint Connector_JST:JST_XH_S3B-XH-SM4-TB_1x03-1MP_P2.50mm_Horizontal -> Connector_PinHeader_2.54mm:PinHeader_1x03_P2.54mm_Vertical; BOM Comments Conector SMD de 3 pines; requiere housing XHP-3 y terminale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 -> Montaje manual: header THT vertical 1x03, paso 2.54 mm. Exc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; LCSC PN C5306495 -> (none); MPN S3B-XH-SM4-TB(LF)(SN) -> Header generico THT 1x03 P2.54 mm; Manufacturer JST -> Compra manual; Manufacturer Part S3B-XH-SM4-TB(LF)(SN) -> Header generico THT 1x03, P2.54 mm, vertical
- R20: footprint (none) -> Resistor_SMD:R_0603_1608Metric
Connections:
- net +5V: now also J5.1 (Pin_1)
- net GND: now also J5.2 (Pin_2)
- no-connect marks 12 -> 13
